Commit message: GZ: Added simplified option to launch files, in order to allow less elements in sim

File: orion_gz/urdf/orion_gz.urdf.xacro (robot description, xacro)
@@ -7,4 +7,5 @@
     <xacro:property name="gazebo" default="$(arg gazebo)"/>
     <xacro:property name="ros2_control" default="$(arg ros2_control)"/>
+    <xacro:property name="simplified" default="true"/>
     <!-- For colors consider mdf, transparent or pla -->
     <xacro:property name="color" default="mdf"/>

Commit message: GZ: Adding new world, updating world params and adding motor param

File: orion_gz/urdf/orion_gz.urdf.xacro (robot description, xacro)
@@ -8,4 +8,5 @@
     <xacro:property name="ros2_control" default="$(arg ros2_control)"/>
     <xacro:property name="simplified" default="true"/>
+    <xacro:property name="motor" value="100"/>
     <!-- For colors consider mdf, transparent or pla -->
     <xacro:property name="color" default="mdf"/>

Commit message: READMEs: Adding new general readme and package readme, with resources

File: orion_gz/urdf/orion_gz.urdf.xacro (robot description, xacro)
@@ -10,5 +10,5 @@
     <xacro:property name="motor" value="100"/>
     <!-- For colors consider mdf, transparent or pla -->
-    <xacro:property name="color" default="mdf"/>
+    <xacro:property name="color" default="pla"/>
     <!-- Include other files -->
     <xacro:include filename="$(find orion_description)/urdf/include/orion_materials.urdf.xacro"/>
