Commit message: General: Updated READMes |GZ: Updated configs for simulation | Docker: Added a devcontainer for sim applications

File: orion_gz/urdf/include/orion_gz_actuators.urdf.xacro (robot description, xacro)
@@ -90,4 +90,11 @@
             </plugin>
         </gazebo>
+        <gazebo>
+            <plugin filename="gz-sim-joint-state-publisher-system"
+                name="gz::sim::systems::JointStatePublisher">
+                <joint_name>caster_middle_2_joint</joint_name>
+                <joint_name>caster_wheel_2_joint</joint_name>
+            </plugin>
+        </gazebo>
     </xacro:unless>
     <xacro:if value="${ros2_control}">
@@ -134,4 +141,12 @@
             </joint>
         </xacro:if>
+            <joint name="caster_middle_2_joint">
+                <state_interface name="position"/>
+                <state_interface name="velocity"/>
+            </joint>
+            <joint name="caster_wheel_2_joint">
+                <state_interface name="position"/>
+                <state_interface name="velocity"/>
+            </joint>
         </ros2_control>
         <gazebo>
@@ -140,11 +155,4 @@
             </plugin>
         </gazebo>
-        <gazebo>
-            <plugin filename="gz-sim-joint-state-publisher-system"
-                name="gz::sim::systems::JointStatePublisher">
-                <joint_name>caster_middle_2_joint</joint_name>
-                <joint_name>caster_wheel_2_joint</joint_name>
-            </plugin>
-        </gazebo>
     </xacro:if>
 </robot>

Commit message: GZ: Updating actuators name, updating topis name and refactoring base URDF for conversion

File: orion_gz/urdf/include/orion_gz_actuators.urdf.xacro (robot description, xacro)
@@ -32,5 +32,5 @@
                     filename="gz-sim-joint-position-controller-system"
                     name="gz::sim::systems::JointPositionController">
-                    <joint_name>servo_conn1_joint</joint_name>
+                    <joint_name>servo_conn_1_joint</joint_name>
                     <p_gain>10</p_gain>
                     <i_gain>0.1</i_gain>
@@ -46,5 +46,5 @@
                     filename="gz-sim-joint-position-controller-system"
                     name="gz::sim::systems::JointPositionController">
-                    <joint_name>servo_conn2_joint</joint_name>
+                    <joint_name>servo_conn_2_joint</joint_name>
                     <p_gain>10</p_gain>
                     <i_gain>0.1</i_gain>
@@ -82,6 +82,6 @@
                 <joint_name>caster_wheel_2_joint</joint_name>
             <xacro:if value="${servo}">
-                <joint_name>servo_conn1_joint</joint_name>
-                <joint_name>servo_conn2_joint</joint_name>
+                <joint_name>servo_conn_1_joint</joint_name>
+                <joint_name>servo_conn_2_joint</joint_name>
             </xacro:if>
             <xacro:if value="${camera == 'a010' and g_mov}">
@@ -120,5 +120,5 @@
             </joint>
         <xacro:if value="${servo}">
-            <joint name="servo_conn1_joint">
+            <joint name="servo_conn_1_joint">
                 <command_interface name="position" />
                 <command_interface name="velocity" />
@@ -126,5 +126,5 @@
                 <state_interface name="velocity" />
             </joint>
-            <joint name="servo_conn2_joint">
+            <joint name="servo_conn_2_joint">
                 <command_interface name="position" />
                 <command_interface name="velocity" />

File: orion_gz/urdf/include/orion_gz_sensors.urdf.xacro (robot description, xacro)
@@ -332,5 +332,5 @@
                 </plugin>
             </gazebo>
-            <gazebo reference="imu">
+            <gazebo reference="g_mov_imu">
                 <sensor name="imu_sensor" type="imu">
                     <always_on>1</always_on>

File: orion_gz/urdf/orion_gz.urdf.xacro (robot description, xacro)
@@ -1,4 +1,19 @@
 <?xml version="1.0"?>
+<!-- @file orion_gz.urdf.xacro
+     @brief Top-level robot description for ORION simulation in Gazebo Harmonic.
+     Mirrors the argument surface of orion_description/urdf/orion.urdf.xacro and
+     adds the Gazebo-specific sensor/actuator includes when `gazebo` is true. -->
 <robot xmlns:xacro="http://www.ros.org/wiki/xacro" name="orion">
+    <!-- Configurable arguments. Defaults match orion.urdf.xacro to keep the
+         simulation aligned with the real-robot description. -->
+    <xacro:arg name="camera" default="os30a"/>
+    <xacro:arg name="servo" default="true"/>
+    <xacro:arg name="g_mov" default="false"/>
+    <xacro:arg name="rasp" default="rpi5"/>
+    <xacro:arg name="gazebo" default="true"/>
+    <xacro:arg name="ros2_control" default="false"/>
+    <xacro:arg name="simplified" default="false"/>
+    <xacro:arg name="motor" default="100"/>
+    <xacro:arg name="color" default="gold"/>
     <xacro:property name="camera" default="$(arg camera)"/>
     <xacro:property name="servo" default="$(arg servo)"/>
@@ -7,14 +22,15 @@
     <xacro:property name="gazebo" default="$(arg gazebo)"/>
     <xacro:property name="ros2_control" default="$(arg ros2_control)"/>
-    <xacro:property name="simplified" default="true"/>
-    <xacro:property name="motor" value="100"/>
-    <!-- For colors consider mdf, transparent or pla -->
-    <xacro:property name="color" default="pla"/>
-    <!-- Include other files -->
+    <xacro:property name="simplified" default="$(arg simplified)"/>
+    <xacro:property name="motor" default="$(arg motor)"/>
+    <xacro:property name="color" default="$(arg color)"/>
+    <!-- Include shared description files from orion_description -->
     <xacro:include filename="$(find orion_description)/urdf/include/orion_materials.urdf.xacro"/>
     <xacro:include filename="$(find orion_description)/urdf/include/orion_macros.urdf.xacro"/>
+    <xacro:include filename="$(find orion_description)/urdf/include/orion_g_mov.urdf.xacro"/>
     <xacro:include filename="$(find orion_description)/urdf/include/orion_base.urdf.xacro"/>
     <xacro:include filename="$(find orion_description)/urdf/include/orion_arms.urdf.xacro"/>
     <xacro:include filename="$(find orion_description)/urdf/include/orion_cameras.urdf.xacro"/>
+    <!-- Gazebo-specific sensor and actuator plugin tags -->
     <xacro:if value="${gazebo}">
         <xacro:include filename="$(find orion_gz)/urdf/include/orion_gz_sensors.urdf.xacro"/>
